File: Shaker.kicad_sch (KiCad schematic)
At the start: 26 parts

Commit message: huellas creadas
Parts:
- GNDtrans1: renamed from GNDtrans; footprint (none) -> Connector_Wire:SolderWire-0.5sqmm_1x01_D0.9mm_OD2.3mm
- In1trans1: renamed from In1trans; footprint (none) -> Connector_Wire:SolderWire-0.5sqmm_1x01_D0.9mm_OD2.3mm
- In2trans1: renamed from In2trans; footprint (none) -> Connector_Wire:SolderWire-0.5sqmm_1x01_D0.9mm_OD2.3mm
- JackL1: renamed from JackL; footprint (none) -> Connector_Wire:SolderWire-0.5sqmm_1x01_D0.9mm_OD2.3mm
- JackR1: renamed from JackR; footprint (none) -> Connector_Wire:SolderWire-0.5sqmm_1x01_D0.9mm_OD2.3mm
- Jackgnd1: renamed from Jackgnd; footprint (none) -> Connector_Wire:SolderWire-0.5sqmm_1x01_D0.9mm_OD2.3mm
- Jackmic1: renamed from Jackmic; footprint (none) -> Connector_Wire:SolderWire-0.5sqmm_1x01_D0.9mm_OD2.3mm
- Led1: renamed from D?; footprint LED_THT:LED_D5.0mm_IRGrey -> LED_THT:LED_D2.0mm_W4.0mm_H2.8mm_FlatTop
- Speaker+1: renamed from Speaker+; footprint (none) -> Connector_Wire:SolderWire-0.5sqmm_1x01_D0.9mm_OD2.3mm
- Speaker-1: renamed from Speaker-; footprint (none) -> Connector_Wire:SolderWire-0.5sqmm_1x01_D0.9mm_OD2.3mm
- renumbered D to D1, U to U1
